Commit message: e

File: description/robot_core.xacro (robot description, xacro)
@@ -26,5 +26,5 @@
             <origin xyz="0.15 0.0 0.0"/>
             <geometry>
-                <<box size="0.1 0.2 0.2"/>
+                <box size="0.1 0.2 0.2"/>
             </geometry>
         </visual>

Commit message: d

File: description/robot_core.xacro (robot description, xacro)
@@ -18,5 +18,5 @@
     <link name="base_link">
     </link>
-    <joint name="chassis_joiny" type="revolute">
+    <joint name="chassis_joiny" type="fixed">
         <parent link="base_link"/>
         <child link="chassis"/>

Commit message: s

File: description/robot_core.xacro (robot description, xacro)
@@ -24,5 +24,5 @@
     <link name="chassis">
         <visual>
-            <origin xyz="0.15 0.0 0.0"/>
+            <origin xyz="0.0 0.0 0.0"/>
             <geometry>
                 <box size="0.1 0.2 0.2"/>

Commit message: d

File: description/robot_core.xacro (robot description, xacro)
@@ -26,5 +26,5 @@
             <origin xyz="0.0 0.0 0.0"/>
             <geometry>
-                <box size="0.1 0.2 0.2"/>
+                <box size="0.2 0.1 0.2"/>
             </geometry>
         </visual>

Commit message: d

File: description/robot_core.xacro (robot description, xacro)
@@ -26,5 +26,5 @@
             <origin xyz="0.0 0.0 0.0"/>
             <geometry>
-                <box size="0.2 0.1 0.2"/>
+                <box size="1.2 0.1 0.1"/>
             </geometry>
         </visual>

Commit message: d

File: description/robot_core.xacro (robot description, xacro)
@@ -26,5 +26,5 @@
             <origin xyz="0.0 0.0 0.0"/>
             <geometry>
-                <box size="1.2 0.1 0.1"/>
+                <box size="0.2 0.1 0.2"/>
             </geometry>
         </visual>

Commit message: w

File: description/robot_core.xacro (robot description, xacro)
@@ -16,6 +16,8 @@
         <color rgba="1 0 0 1" />
     </material>
+    <!--Base link-->
     <link name="base_link">
     </link>
+    <!--Chassis link-->
     <joint name="chassis_joiny" type="fixed">
         <parent link="base_link"/>
@@ -30,3 +32,18 @@
         </visual>
     </link>
+    <!--Left front Wheel -->
+    <joint name="left_front_wheel" type="continuous">
+        <parent link="base_link"/>
+        <child link="Left_wheel"/>
+        <origin xyz="0.0 0.175 0.0" rpy="-${pi/2} 0.0 0.0"/>
+        <axis xyz="0.0 0.0 1.0"/>
+    </joint>
+    <link name="Left_wheel">
+        <visual>
+            <geometry>
+                <cylinder radius="0.065" length="0.03"/>
+            </geometry>
+            <material name="white">
+        </visual>
+    </link>
 </robot>

Commit message: f

File: description/robot_core.xacro (robot description, xacro)
@@ -20,5 +20,5 @@
     </link>
     <!--Chassis link-->
-    <joint name="chassis_joiny" type="fixed">
+    <joint name="chassis_joint" type="fixed">
         <parent link="base_link"/>
         <child link="chassis"/>
@@ -44,5 +44,5 @@
                 <cylinder radius="0.065" length="0.03"/>
             </geometry>
-            <material name="white">
+            <material name="white"/>
         </visual>
     </link>

Commit message: d

File: description/robot_core.xacro (robot description, xacro)
@@ -28,5 +28,5 @@
             <origin xyz="0.0 0.0 0.0"/>
             <geometry>
-                <box size="0.2 0.1 0.2"/>
+                <box size="0.2 0.2 0.01"/>
             </geometry>
         </visual>
@@ -37,5 +37,5 @@
         <child link="Left_wheel"/>
         <origin xyz="0.0 0.175 0.0" rpy="-${pi/2} 0.0 0.0"/>
-        <axis xyz="0.0 0.0 1.0"/>
+        <axis xyz="0.0 0.0 -1.0"/>
     </joint>
     <link name="Left_wheel">

Commit message: correcting box shape

File: description/robot_core.xacro (robot description, xacro)
@@ -28,5 +28,5 @@
             <origin xyz="0.0 0.0 0.0"/>
             <geometry>
-                <box size="0.2 0.2 0.01"/>
+                <box size="0.241 0.195 0.2"/>
             </geometry>
         </visual>

Commit message: fixing position of wheel and orgin of box

File: description/robot_core.xacro (robot description, xacro)
@@ -26,5 +26,5 @@
     <link name="chassis">
         <visual>
-            <origin xyz="0.0 0.0 0.0"/>
+            <origin xyz="0.0 0.0 0.2"/>
             <geometry>
                 <box size="0.241 0.195 0.2"/>
@@ -36,5 +36,5 @@
         <parent link="base_link"/>
         <child link="Left_wheel"/>
-        <origin xyz="0.0 0.175 0.0" rpy="-${pi/2} 0.0 0.0"/>
+        <origin xyz="-0.349 0.0 0.0" rpy="-${pi/2} 0.0 0.0"/>
         <axis xyz="0.0 0.0 -1.0"/>
     </joint>

Commit message: box

File: description/robot_core.xacro (robot description, xacro)
@@ -26,5 +26,5 @@
     <link name="chassis">
         <visual>
-            <origin xyz="0.0 0.0 0.2"/>
+            <origin xyz="0.0 0.0 0.015"/>
             <geometry>
                 <box size="0.241 0.195 0.2"/>
@@ -37,5 +37,5 @@
         <child link="Left_wheel"/>
         <origin xyz="-0.349 0.0 0.0" rpy="-${pi/2} 0.0 0.0"/>
-        <axis xyz="0.0 0.0 -1.0"/>
+        <axis xyz="0.0 0.0 -0.05"/>
     </joint>
     <link name="Left_wheel">

Commit message: box

File: description/robot_core.xacro (robot description, xacro)
@@ -26,5 +26,5 @@
     <link name="chassis">
         <visual>
-            <origin xyz="0.0 0.0 0.015"/>
+            <origin xyz="0.0 0.0 0.035"/>
             <geometry>
                 <box size="0.241 0.195 0.2"/>
@@ -37,5 +37,5 @@
         <child link="Left_wheel"/>
         <origin xyz="-0.349 0.0 0.0" rpy="-${pi/2} 0.0 0.0"/>
-        <axis xyz="0.0 0.0 -0.05"/>
+        <axis xyz="0.0 0.0 -0.035"/>
     </joint>
     <link name="Left_wheel">

Commit message: origin

File: description/robot_core.xacro (robot description, xacro)
@@ -42,5 +42,5 @@
         <visual>
             <geometry>
-                <cylinder radius="0.065" length="0.03"/>
+                <cylinder radius="0.0285" length="0.0"/>
             </geometry>
             <material name="white"/>

Commit message: wheel

File: description/robot_core.xacro (robot description, xacro)
@@ -36,11 +36,11 @@
         <parent link="base_link"/>
         <child link="Left_wheel"/>
-        <origin xyz="-0.349 0.0 0.0" rpy="-${pi/2} 0.0 0.0"/>
-        <axis xyz="0.0 0.0 -0.035"/>
+        <origin xyz="-0.149 0.0 0.0" rpy="-${pi/2} 0.0 0.0"/>
+        <axis xyz="0.0 0.0 1"/>
     </joint>
     <link name="Left_wheel">
         <visual>
             <geometry>
-                <cylinder radius="0.0285" length="0.0"/>
+                <cylinder radius="0.0285" length="0.025"/>
             </geometry>
             <material name="white"/>

Commit message: box

File: description/robot_core.xacro (robot description, xacro)
@@ -26,5 +26,5 @@
     <link name="chassis">
         <visual>
-            <origin xyz="0.0 0.0 0.035"/>
+            <origin xyz="0.0 0.0 0.078"/>
             <geometry>
                 <box size="0.241 0.195 0.2"/>
@@ -36,5 +36,5 @@
         <parent link="base_link"/>
         <child link="Left_wheel"/>
-        <origin xyz="-0.149 0.0 0.0" rpy="-${pi/2} 0.0 0.0"/>
+        <origin xyz="-0.055 0.195 0.0" rpy="-${pi/2} 0.0 0.0"/>
         <axis xyz="0.0 0.0 1"/>
     </joint>

Commit message: d

File: description/robot_core.xacro (robot description, xacro)
@@ -36,5 +36,5 @@
         <parent link="base_link"/>
         <child link="Left_wheel"/>
-        <origin xyz="-0.055 0.195 0.0" rpy="-${pi/2} 0.0 0.0"/>
+        <origin xyz="-0.055 0.085 0.0" rpy="-${pi/2} 0.0 0.0"/>
         <axis xyz="0.0 0.0 1"/>
     </joint>

Commit message: d

File: description/robot_core.xacro (robot description, xacro)
@@ -36,5 +36,5 @@
         <parent link="base_link"/>
         <child link="Left_wheel"/>
-        <origin xyz="-0.055 0.085 0.0" rpy="-${pi/2} 0.0 0.0"/>
+        <origin xyz="-0.055 0.095 0.0" rpy="-${pi/2} 0.0 0.0"/>
         <axis xyz="0.0 0.0 1"/>
     </joint>

Commit message: might be final hange to fron left wheel

File: description/robot_core.xacro (robot description, xacro)
@@ -36,5 +36,5 @@
         <parent link="base_link"/>
         <child link="Left_wheel"/>
-        <origin xyz="-0.055 0.095 0.0" rpy="-${pi/2} 0.0 0.0"/>
+        <origin xyz="-0.055 0.105 0.0" rpy="-${pi/2} 0.0 0.0"/>
         <axis xyz="0.0 0.0 1"/>
     </joint>

Commit message: d

File: description/robot_core.xacro (robot description, xacro)
@@ -36,5 +36,5 @@
         <parent link="base_link"/>
         <child link="Left_wheel"/>
-        <origin xyz="-0.055 0.105 0.0" rpy="-${pi/2} 0.0 0.0"/>
+        <origin xyz="-0.050 0.105 0.0" rpy="-${pi/2} 0.0 0.0"/>
         <axis xyz="0.0 0.0 1"/>
     </joint>

Commit message: d

File: description/robot_core.xacro (robot description, xacro)
@@ -36,5 +36,5 @@
         <parent link="base_link"/>
         <child link="Left_wheel"/>
-        <origin xyz="-0.050 0.105 0.0" rpy="-${pi/2} 0.0 0.0"/>
+        <origin xyz="-0.060 0.105 0.0" rpy="-${pi/2} 0.0 0.0"/>
         <axis xyz="0.0 0.0 1"/>
     </joint>

Commit message: final change to left_front_wheel

File: description/robot_core.xacro (robot description, xacro)
@@ -36,5 +36,5 @@
         <parent link="base_link"/>
         <child link="Left_wheel"/>
-        <origin xyz="-0.060 0.105 0.0" rpy="-${pi/2} 0.0 0.0"/>
+        <origin xyz="-0.075 0.109 0.0" rpy="-${pi/2} 0.0 0.0"/>
         <axis xyz="0.0 0.0 1"/>
     </joint>

Commit message: front right wheel added

File: description/robot_core.xacro (robot description, xacro)
@@ -47,3 +47,18 @@
         </visual>
     </link>
+    <!--Right front Wheel -->
+    <joint name="left_front_wheel" type="continuous">
+        <parent link="base_link"/>
+        <child link="Left_wheel"/>
+        <origin xyz="0.075 0.109 0.0" rpy="-${pi/2} 0.0 0.0"/>
+        <axis xyz="0.0 0.0 1"/>
+    </joint>
+    <link name="Left_wheel">
+        <visual>
+            <geometry>
+                <cylinder radius="0.0285" length="0.025"/>
+            </geometry>
+            <material name="white"/>
+        </visual>
+    </link>
 </robot>

Commit message: right wheel fixed

File: description/robot_core.xacro (robot description, xacro)
@@ -50,9 +50,9 @@
     <joint name="left_front_wheel" type="continuous">
         <parent link="base_link"/>
-        <child link="Left_wheel"/>
+        <child link="Right_wheel"/>
         <origin xyz="0.075 0.109 0.0" rpy="-${pi/2} 0.0 0.0"/>
         <axis xyz="0.0 0.0 1"/>
     </joint>
-    <link name="Left_wheel">
+    <link name="Right_wheel">
         <visual>
             <geometry>

Commit message: Right wheel named fixed in xml

File: description/robot_core.xacro (robot description, xacro)
@@ -48,5 +48,5 @@
     </link>
     <!--Right front Wheel -->
-    <joint name="left_front_wheel" type="continuous">
+    <joint name="Right_front_wheel" type="continuous">
         <parent link="base_link"/>
         <child link="Right_wheel"/>

Commit message: changing front right to left rear

File: description/robot_core.xacro (robot description, xacro)
@@ -44,15 +44,15 @@
                 <cylinder radius="0.0285" length="0.025"/>
             </geometry>
-            <material name="white"/>
+            <material name="Blue"/>
         </visual>
     </link>
     <!--Right front Wheel -->
-    <joint name="Right_front_wheel" type="continuous">
+    <joint name="Left_Rear_wheel" type="continuous">
         <parent link="base_link"/>
-        <child link="Right_wheel"/>
+        <child link="Left_rear_wheel"/>
         <origin xyz="0.075 0.109 0.0" rpy="-${pi/2} 0.0 0.0"/>
         <axis xyz="0.0 0.0 1"/>
     </joint>
-    <link name="Right_wheel">
+    <link name="Right_rear_wheel">
         <visual>
             <geometry>

Commit message: d

File: description/robot_core.xacro (robot description, xacro)
@@ -33,11 +33,11 @@
     </link>
     <!--Left front Wheel -->
-    <joint name="left_front_wheel" type="continuous">
+    <joint name="Left_Front_wheel" type="continuous">
         <parent link="base_link"/>
-        <child link="Left_wheel"/>
+        <child link="Left_Front_wheel"/>
         <origin xyz="-0.075 0.109 0.0" rpy="-${pi/2} 0.0 0.0"/>
         <axis xyz="0.0 0.0 1"/>
     </joint>
-    <link name="Left_wheel">
+    <link name="Left_Front_wheel">
         <visual>
             <geometry>
@@ -50,9 +50,9 @@
     <joint name="Left_Rear_wheel" type="continuous">
         <parent link="base_link"/>
-        <child link="Left_rear_wheel"/>
+        <child link="Left_Rear_wheel"/>
         <origin xyz="0.075 0.109 0.0" rpy="-${pi/2} 0.0 0.0"/>
         <axis xyz="0.0 0.0 1"/>
     </joint>
-    <link name="Right_rear_wheel">
+    <link name="Left_Rear_wheel">
         <visual>
             <geometry>

Commit message: Left rear and front wheels added

File: description/robot_core.xacro (robot description, xacro)
@@ -32,9 +32,39 @@
         </visual>
     </link>
+    <!--Right front Wheel -->
+    <joint name="Right_Front_wheel" type="continuous">
+        <parent link="base_link"/>
+        <child link="Right_Front_wheel"/>
+        <origin xyz="-0.075 0.109 0.0" rpy="-${pi/2} 0.0 0.0"/>
+        <axis xyz="0.0 0.0 1"/>
+    </joint>
+    <link name="Right_Front_wheel">
+        <visual>
+            <geometry>
+                <cylinder radius="0.0285" length="0.025"/>
+            </geometry>
+            <material name="Blue"/>
+        </visual>
+    </link>
+    <!--Right Rear Wheel -->
+    <joint name="Right_Rear_wheel" type="continuous">
+        <parent link="base_link"/>
+        <child link="Right_Rear_wheel"/>
+        <origin xyz="0.075 0.109 0.0" rpy="-${pi/2} 0.0 0.0"/>
+        <axis xyz="0.0 0.0 1"/>
+    </joint>
+    <link name="Right_Rear_wheel">
+        <visual>
+            <geometry>
+                <cylinder radius="0.0285" length="0.025"/>
+            </geometry>
+            <material name="white"/>
+        </visual>
+    </link>
     <!--Left front Wheel -->
-    <joint name="Left_Front_wheel" type="continuous">
+<joint name="left_Front_wheel" type="continuous">
         <parent link="base_link"/>
         <child link="Left_Front_wheel"/>
-        <origin xyz="-0.075 0.109 0.0" rpy="-${pi/2} 0.0 0.0"/>
+        <origin xyz="-0.075 -0.109 0.0" rpy="-${pi/2} 0.0 0.0"/>
         <axis xyz="0.0 0.0 1"/>
     </joint>
@@ -47,9 +77,9 @@
         </visual>
     </link>
-    <!--Right front Wheel -->
+   <!--Left Rear Wheel -->
     <joint name="Left_Rear_wheel" type="continuous">
         <parent link="base_link"/>
         <child link="Left_Rear_wheel"/>
-        <origin xyz="0.075 0.109 0.0" rpy="-${pi/2} 0.0 0.0"/>
+        <origin xyz="0.075 -0.109 0.0" rpy="-${pi/2} 0.0 0.0"/>
         <axis xyz="0.0 0.0 1"/>
     </joint>

Commit message: caster wheel

File: description/robot_core.xacro (robot description, xacro)
@@ -92,3 +92,17 @@
         </visual>
     </link>
+     <!--Caster Wheel Link-->
+     <joint name="caster_wheel_link" type="fixed">
+        <parent link="chassis"/>
+        <child link="caster_wheel"/>
+        <origin xyz="0.0 0.0 0.078"/>
+     </joint>
+     <link name="caster_wheel">
+        <visual>
+            <geometry>
+                <sphere radius="0.05"/>
+            </geometry>
+            <material name="orange"/>
+        </visual>
+     </link>
 </robot>

Commit message: d

File: description/robot_core.xacro (robot description, xacro)
@@ -96,5 +96,5 @@
         <parent link="chassis"/>
         <child link="caster_wheel"/>
-        <origin xyz="0.0 0.0 0.078"/>
+        <origin xyz="0.0 0.0 -0.108"/>
      </joint>
      <link name="caster_wheel">

Commit message: d

File: description/robot_core.xacro (robot description, xacro)
@@ -96,5 +96,5 @@
         <parent link="chassis"/>
         <child link="caster_wheel"/>
-        <origin xyz="0.0 0.0 -0.108"/>
+        <origin xyz="0.0 0.0 -0.1"/>
      </joint>
      <link name="caster_wheel">

Commit message: d

File: description/robot_core.xacro (robot description, xacro)
@@ -96,5 +96,5 @@
         <parent link="chassis"/>
         <child link="caster_wheel"/>
-        <origin xyz="0.0 0.0 -0.1"/>
+        <origin xyz="0.0 0.0 -0.08"/>
      </joint>
      <link name="caster_wheel">

Commit message: d

File: description/robot_core.xacro (robot description, xacro)
@@ -96,5 +96,5 @@
         <parent link="chassis"/>
         <child link="caster_wheel"/>
-        <origin xyz="0.0 0.0 -0.08"/>
+        <origin xyz="0.0 0.0 -0.01"/>
      </joint>
      <link name="caster_wheel">

Commit message: d

File: description/robot_core.xacro (robot description, xacro)
@@ -96,5 +96,5 @@
         <parent link="chassis"/>
         <child link="caster_wheel"/>
-        <origin xyz="0.0 0.0 -0.01"/>
+        <origin xyz="0.0 0.0 -0.02"/>
      </joint>
      <link name="caster_wheel">

Commit message: changing position of caster wheel to match

File: description/robot_core.xacro (robot description, xacro)
@@ -28,5 +28,5 @@
             <origin xyz="0.0 0.0 0.078"/>
             <geometry>
-                <box size="0.241 0.195 0.2"/>
+                <box size="0.241 0.195 0.285"/>
             </geometry>
         </visual>
@@ -96,10 +96,10 @@
         <parent link="chassis"/>
         <child link="caster_wheel"/>
-        <origin xyz="0.0 0.0 -0.02"/>
+        <origin xyz="0.0 0.0 -0.0285"/>
      </joint>
      <link name="caster_wheel">
         <visual>
             <geometry>
-                <sphere radius="0.05"/>
+                <sphere radius="0.0285"/>
             </geometry>
             <material name="orange"/>

Commit message: position

File: description/robot_core.xacro (robot description, xacro)
@@ -26,7 +26,7 @@
     <link name="chassis">
         <visual>
-            <origin xyz="0.0 0.0 0.078"/>
+            <origin xyz="0.0 0.0 0.285"/>
             <geometry>
-                <box size="0.241 0.195 0.285"/>
+                <box size="0.241 0.195 0.2"/>
             </geometry>
         </visual>

Commit message: p

File: description/robot_core.xacro (robot description, xacro)
@@ -26,5 +26,5 @@
     <link name="chassis">
         <visual>
-            <origin xyz="0.0 0.0 0.285"/>
+            <origin xyz="0.0 0.0 0.0285"/>
             <geometry>
                 <box size="0.241 0.195 0.2"/>

Commit message: p

File: description/robot_core.xacro (robot description, xacro)
@@ -26,5 +26,5 @@
     <link name="chassis">
         <visual>
-            <origin xyz="0.0 0.0 0.0285"/>
+            <origin xyz="0.0 0.0 0.09"/>
             <geometry>
                 <box size="0.241 0.195 0.2"/>

Commit message: p

File: description/robot_core.xacro (robot description, xacro)
@@ -96,5 +96,5 @@
         <parent link="chassis"/>
         <child link="caster_wheel"/>
-        <origin xyz="0.0 0.0 -0.0285"/>
+        <origin xyz="0.0 0.0 -0.0235"/>
      </joint>
      <link name="caster_wheel">

Commit message: p

File: description/robot_core.xacro (robot description, xacro)
@@ -96,5 +96,5 @@
         <parent link="chassis"/>
         <child link="caster_wheel"/>
-        <origin xyz="0.0 0.0 -0.0235"/>
+        <origin xyz="0.0 0.0 -0.02"/>
      </joint>
      <link name="caster_wheel">

Commit message: p

File: description/robot_core.xacro (robot description, xacro)
@@ -96,5 +96,5 @@
         <parent link="chassis"/>
         <child link="caster_wheel"/>
-        <origin xyz="0.0 0.0 -0.02"/>
+        <origin xyz="0.0 0.0 -0.015"/>
      </joint>
      <link name="caster_wheel">

Commit message: p

File: description/robot_core.xacro (robot description, xacro)
@@ -96,5 +96,5 @@
         <parent link="chassis"/>
         <child link="caster_wheel"/>
-        <origin xyz="0.0 0.0 -0.015"/>
+        <origin xyz="0.0 0.0 -0.01"/>
      </joint>
      <link name="caster_wheel">

Commit message: p

File: description/robot_core.xacro (robot description, xacro)
@@ -96,5 +96,5 @@
         <parent link="chassis"/>
         <child link="caster_wheel"/>
-        <origin xyz="0.0 0.0 -0.01"/>
+        <origin xyz="0.0 0.0 0.0"/>
      </joint>
      <link name="caster_wheel">

Commit message: change wheels face front

File: description/robot_core.xacro (robot description, xacro)
@@ -32,9 +32,24 @@
         </visual>
     </link>
-    <!--Right front Wheel -->
+    <!--Right Rear Wheel -->
+    <joint name="Right_Rear_wheel" type="continuous">
+        <parent link="base_link"/>
+        <child link="Right_Rear_wheel"/>
+        <origin xyz="-0.075 0.109 0.0" rpy="-${pi/2} 0.0 0.0"/>
+        <axis xyz="0.0 0.0 1"/>
+    </joint>
+    <link name="Right_Rear_wheel">
+        <visual>
+            <geometry>
+                <cylinder radius="0.0285" length="0.025"/>
+            </geometry>
+            <material name="Blue"/>
+        </visual>
+    </link>
+    <!--Right Front Wheel -->
     <joint name="Right_Front_wheel" type="continuous">
         <parent link="base_link"/>
         <child link="Right_Front_wheel"/>
-        <origin xyz="-0.075 0.109 0.0" rpy="-${pi/2} 0.0 0.0"/>
+        <origin xyz="0.075 0.109 0.0" rpy="-${pi/2} 0.0 0.0"/>
         <axis xyz="0.0 0.0 1"/>
     </joint>
@@ -44,30 +59,15 @@
                 <cylinder radius="0.0285" length="0.025"/>
             </geometry>
-            <material name="Blue"/>
-        </visual>
-    </link>
-    <!--Right Rear Wheel -->
-    <joint name="Right_Rear_wheel" type="continuous">
-        <parent link="base_link"/>
-        <child link="Right_Rear_wheel"/>
-        <origin xyz="0.075 0.109 0.0" rpy="-${pi/2} 0.0 0.0"/>
-        <axis xyz="0.0 0.0 1"/>
-    </joint>
-    <link name="Right_Rear_wheel">
-        <visual>
-            <geometry>
-                <cylinder radius="0.0285" length="0.025"/>
-            </geometry>
             <material name="white"/>
         </visual>
     </link>
-    <!--Left front Wheel -->
-<joint name="left_Front_wheel" type="continuous">
+    <!--Left Rear Wheel -->
+<joint name="left_Rear_wheel" type="continuous">
         <parent link="base_link"/>
-        <child link="Left_Front_wheel"/>
+        <child link="Left_Rear_wheel"/>
         <origin xyz="-0.075 -0.109 0.0" rpy="-${pi/2} 0.0 0.0"/>
         <axis xyz="0.0 0.0 1"/>
     </joint>
-    <link name="Left_Front_wheel">
+    <link name="Left_Rear_wheel">
         <visual>
             <geometry>
@@ -77,12 +77,12 @@
         </visual>
     </link>
-   <!--Left Rear Wheel -->
-    <joint name="Left_Rear_wheel" type="continuous">
+   <!--Left Front Wheel -->
+    <joint name="Left_Front_wheel" type="continuous">
         <parent link="base_link"/>
-        <child link="Left_Rear_wheel"/>
+        <child link="Left_Front_wheel"/>
         <origin xyz="0.075 -0.109 0.0" rpy="-${pi/2} 0.0 0.0"/>
         <axis xyz="0.0 0.0 1"/>
     </joint>
-    <link name="Left_Rear_wheel">
+    <link name="Left_Front_wheel">
         <visual>
             <geometry>
