Commit message: collision

File: description/robot_core.xacro (robot description, xacro)
@@ -31,4 +31,10 @@
             </geometry>
         </visual>
+        <collision>
+            <origin xyz="0.0 0.0 0.09"/>
+            <geometry>
+                <box size="0.241 0.195 0.2"/>
+            </geometry>
+        </collision>
     </link>
     <!--Right Rear Wheel -->
@@ -46,4 +52,9 @@
             <material name="Blue"/>
         </visual>
+        <collision>
+            <geometry>
+                <cylinder radius="0.0285" length="0.025"/>
+            </geometry>
+        </collision>
     </link>
     <!--Right Front Wheel -->
@@ -61,4 +72,9 @@
             <material name="white"/>
         </visual>
+        <collision>
+            <geometry>
+                <cylinder radius="0.0285" length="0.025"/>
+            </geometry>
+        </collision>
     </link>
     <!--Left Rear Wheel -->
@@ -76,4 +92,9 @@
             <material name="Blue"/>
         </visual>
+        <collision>
+            <geometry>
+                <cylinder radius="0.0285" length="0.025"/>
+            </geometry>
+        </collision>
     </link>
    <!--Left Front Wheel -->
@@ -91,4 +112,9 @@
             <material name="white"/>
         </visual>
+        <collision>
+            <geometry>
+                <cylinder radius="0.0285" length="0.025"/>
+            </geometry>
+        </collision>
     </link>
      <!--Caster Wheel Link-->
@@ -105,4 +131,9 @@
             <material name="orange"/>
         </visual>
+        <collision>
+            <geometry>
+                <sphere radius="0.0285"/>
+            </geometry>
+        </collision>
      </link>
 </robot>

Commit message: interial added

File: description/robot_core.xacro (robot description, xacro)
@@ -1,4 +1,5 @@
 <?xml version="1.0"?>
 <robot xmlns:xacro="http://www.ros.org/wiki/xacro"  name="robot">
+    <xacro:include filename="inertial_macros.xacro"/>
 <material name="white">
         <color rgba="1 1 1 1" />
@@ -37,4 +38,7 @@
             </geometry>
         </collision>
+        <xacro:inertial_box mass="0.5" x="0.241" y="0.195" z="0.2">
+            <origin xyz="0.0 0.0 0.09" rpy="0.0 0.0 0.0"/>
+        </xacro:inertial_box>
     </link>
     <!--Right Rear Wheel -->
@@ -57,4 +61,7 @@
             </geometry>
         </collision>
+        <xacro:inertial_cylinder mass="0.1" length="0.025" radius="0.0285">
+            <origin xyz="0.0 0.0 0.0" rpy="0.0 0.0 0.0"/>
+        </xacro:inertial_cylinder>
     </link>
     <!--Right Front Wheel -->
@@ -77,4 +84,7 @@
             </geometry>
         </collision>
+        <xacro:inertial_cylinder mass="0.1" length="0.025" radius="0.0285">
+            <origin xyz="0.0 0.0 0.0" rpy="0.0 0.0 0.0"/>
+        </xacro:inertial_cylinder>
     </link>
     <!--Left Rear Wheel -->
@@ -97,4 +107,7 @@
             </geometry>
         </collision>
+        <xacro:inertial_cylinder mass="0.1" length="0.025" radius="0.0285">
+            <origin xyz="0.0 0.0 0.0" rpy="0.0 0.0 0.0"/>
+        </xacro:inertial_cylinder>
     </link>
    <!--Left Front Wheel -->
@@ -117,4 +130,7 @@
             </geometry>
         </collision>
+        <xacro:inertial_cylinder mass="0.1" length="0.025" radius="0.0285">
+            <origin xyz="0.0 0.0 0.0" rpy="0.0 0.0 0.0"/>
+        </xacro:inertial_cylinder>
     </link>
      <!--Caster Wheel Link-->
@@ -136,4 +152,7 @@
             </geometry>
         </collision>
+        <xacro:inertial_sphere mass="0.1" radius="0.0285">
+            <origin xyz="0.0 0.0 0.0" rpy="0.0 0.0 0.0"/>
+        </xacro:inertial_sphere>
      </link>
 </robot>

Commit message: change link name

File: description/robot_core.xacro (robot description, xacro)
@@ -43,5 +43,5 @@
     </link>
     <!--Right Rear Wheel -->
-    <joint name="Right_Rear_wheel" type="continuous">
+    <joint name="Right_Rear_wheel_j" type="continuous">
         <parent link="base_link"/>
         <child link="Right_Rear_wheel"/>

Commit message: fixed joint names for gazeebo

File: description/robot_core.xacro (robot description, xacro)
@@ -43,5 +43,5 @@
     </link>
     <!--Right Rear Wheel -->
-    <joint name="Right_Rear_wheel_j" type="continuous">
+    <joint name="Right_Rear_wheel_joint" type="continuous">
         <parent link="base_link"/>
         <child link="Right_Rear_wheel"/>
@@ -66,5 +66,5 @@
     </link>
     <!--Right Front Wheel -->
-    <joint name="Right_Front_wheel" type="continuous">
+    <joint name="Right_Front_wheel_joint" type="continuous">
         <parent link="base_link"/>
         <child link="Right_Front_wheel"/>
@@ -89,5 +89,5 @@
     </link>
     <!--Left Rear Wheel -->
-<joint name="left_Rear_wheel" type="continuous">
+<joint name="left_Rear_wheel_joint" type="continuous">
         <parent link="base_link"/>
         <child link="Left_Rear_wheel"/>
@@ -112,5 +112,5 @@
     </link>
    <!--Left Front Wheel -->
-    <joint name="Left_Front_wheel" type="continuous">
+    <joint name="Left_Front_wheel_joint" type="continuous">
         <parent link="base_link"/>
         <child link="Left_Front_wheel"/>

Commit message: Gazebo colors

File: description/robot_core.xacro (robot description, xacro)
@@ -42,4 +42,7 @@
         </xacro:inertial_box>
     </link>
+    <gazebo reference="chassis">
+        <material>Gazebo/White</material>
+    </gazebo>
     <!--Right Rear Wheel -->
     <joint name="Right_Rear_wheel_joint" type="continuous">
@@ -65,4 +68,7 @@
         </xacro:inertial_cylinder>
     </link>
+    <gazebo reference="Right_Rear_wheel">
+        <material>Gazebo/Blue</material>
+    </gazebo>
     <!--Right Front Wheel -->
     <joint name="Right_Front_wheel_joint" type="continuous">
@@ -77,5 +83,5 @@
                 <cylinder radius="0.0285" length="0.025"/>
             </geometry>
-            <material name="white"/>
+            <material name="red"/>
         </visual>
         <collision>
@@ -88,4 +94,7 @@
         </xacro:inertial_cylinder>
     </link>
+    <gazebo reference="Right_Front_wheel">
+        <material>Gazebo/Red</material>
+    </gazebo>
     <!--Left Rear Wheel -->
 <joint name="left_Rear_wheel_joint" type="continuous">
@@ -111,4 +120,7 @@
         </xacro:inertial_cylinder>
     </link>
+    <gazebo reference="Left_Rear_wheel">
+        <material>Gazebo/Blue</material>
+    </gazebo>
    <!--Left Front Wheel -->
     <joint name="Left_Front_wheel_joint" type="continuous">
@@ -123,5 +135,5 @@
                 <cylinder radius="0.0285" length="0.025"/>
             </geometry>
-            <material name="white"/>
+            <material name="red"/>
         </visual>
         <collision>
@@ -134,4 +146,7 @@
         </xacro:inertial_cylinder>
     </link>
+    <gazebo reference="Left_Front_wheel">
+        <material>Gazebo/Red</material>
+    </gazebo>
      <!--Caster Wheel Link-->
      <joint name="caster_wheel_link" type="fixed">
@@ -156,3 +171,6 @@
         </xacro:inertial_sphere>
      </link>
+     <gazebo reference="caster_wheel">
+        <material>Gazebo/Black</material>
+    </gazebo>
 </robot>
