Commit message: d

File: description/lidar.xacro (robot description, xacro)
@@ -4,5 +4,5 @@
         <parent link="chassis"/>
         <child link="laser_frame"/>
-        <origin xyz="0.2 0.0 0.21" rpy="0 0 0"/>
+        <origin xyz="0.1 0.0 0.21" rpy="0 0 0"/>
     </joint>
     <link name="laser_frame">

Commit message: fixing lidar position

File: description/lidar.xacro (robot description, xacro)
@@ -4,5 +4,5 @@
         <parent link="chassis"/>
         <child link="laser_frame"/>
-        <origin xyz="0.1 0.0 0.21" rpy="0 0 0"/>
+        <origin xyz="0.1 0.0 0.2" rpy="0 0 0"/>
     </joint>
     <link name="laser_frame">

Commit message: adding gazebo lidar color

File: description/lidar.xacro (robot description, xacro)
@@ -22,3 +22,6 @@
         </xacro:inertial_cylinder>
     </link>
+    <gazebo reference="Right_Rear_wheel">
+        <material>Gazebo/red</material>
+    </gazebo>
 </robot>

Commit message: simulated sensor

File: description/lidar.xacro (robot description, xacro)
@@ -23,5 +23,5 @@
     </link>
     <gazebo reference="laser_frame">
-        <material>Gazebo/red</material>
+        <sensor name="laser" type="ray">
     </gazebo>
 </robot>

Commit message: color lidar

File: description/lidar.xacro (robot description, xacro)
@@ -23,4 +23,5 @@
     </link>
     <gazebo reference="laser_frame">
+        <<material>Gazebo/Red</material>
         <sensor name="laser" type="ray">
             <pose> 0 0 0 0 0 0 </pose>

Commit message: d

File: description/lidar.xacro (robot description, xacro)
@@ -23,5 +23,5 @@
     </link>
     <gazebo reference="laser_frame">
-        <<material>Gazebo/Red</material>
+        <material>Gazebo/Red</material>
         <sensor name="laser" type="ray">
             <pose> 0 0 0 0 0 0 </pose>
