Commit message: d

File: description/depth_camera.xacro (robot description, xacro)
@@ -19,5 +19,5 @@
         <origin xyz="0.245 0.0 0.0" rpy="${-pi/2} 0 ${-pi/2}"/>
     </joint>
-    <link name="camera_link_optical" type="fixed">
+    <link name="camera_link_optical" type="fixed"></link>
     <gazebo reference="camera_link">
         <material>Gazebo/Red</material>

Commit message: fix camera link

File: description/depth_camera.xacro (robot description, xacro)
@@ -19,5 +19,5 @@
         <origin xyz="0.245 0.0 0.0" rpy="${-pi/2} 0 ${-pi/2}"/>
     </joint>
-    <link name="camera_link_optical" type="fixed"></link>
+    <link name="camera_link_optical"></link>
     <gazebo reference="camera_link">
         <material>Gazebo/Red</material>

Commit message: c

File: description/depth_camera.xacro (robot description, xacro)
@@ -19,5 +19,5 @@
         <origin xyz="0.245 0.0 0.0" rpy="${-pi/2} 0 ${-pi/2}"/>
     </joint>
-    <link name="camera_link_optical"></link>
+    <link name="camera_link_optical">
     <gazebo reference="camera_link">
         <material>Gazebo/Red</material>

Commit message: a

File: description/depth_camera.xacro (robot description, xacro)
@@ -19,5 +19,5 @@
         <origin xyz="0.245 0.0 0.0" rpy="${-pi/2} 0 ${-pi/2}"/>
     </joint>
-    <link name="camera_link_optical">
+    <link name="camera_link_optical"></link>
     <gazebo reference="camera_link">
         <material>Gazebo/Red</material>
